File: Hardware/Phone/Phone.kicad_sch (KiCad schematic)
At the start: 20 parts, among them J1 UART, J2 JTAG, J3 USB_C_Receptacle_USB2.0_16P, U1 ESP32-S3-WROOM-1, U2 USBLC6-2SC6

Commit message: e ink is done
Parts:
- F1: value 500mA PTC -> 2A PTC
Other:
- added sheet eink Display (display.kicad_sch)
- sheet gsm ports: added DTR, PWRKEY, RX, TX; removed none
Changed lines of the file:
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@@
 	(wire
 		(pts
-			(xy 125.73 143.51) (xy 125.73 151.13)
-		)
-		(stroke
-			(width 0)
-			(type default)
-		)
-	)
-	(wire
-		(pts
 			(xy 127 73.66) (xy 127 74.93)
 		)
@@
 	(wire
 		(pts
-			(xy 125.73 143.51) (xy 124.46 143.51)
-		)
-		(stroke
-			(width 0)
-			(type default)
-		)
-	)
-	(wire
-		(pts
 			(xy 205.74 113.03) (xy 124.46 113.03)
 		)
@@
 	(wire
 		(pts
-			(xy 124.46 146.05) (xy 128.27 146.05)
-		)
-		(stroke
-			(width 0)
-			(type default)
-		)
-	)
-	(wire
-		(pts
 			(xy 251.46 113.03) (xy 251.46 115.57)
 		)
@@
 	(wire
 		(pts
-			(xy 128.27 146.05) (xy 128.27 151.13)
-		)
-		(stroke
-			(width 0)
-			(type default)
-		)
-	)
-	(wire
-		(pts
 			(xy 233.68 113.03) (xy 231.14 110.49)
 		)
@@
 			)
 		)
-		(property "Value" "500mA PTC"
+		(property "Value" "2A PTC"
 			(at 232.41 93.218 90)
 			(effects
@@
 	)
 	(sheet
-		(at 25.4 105.41)
-		(size 22.86 13.97)
+		(at 27.94 99.06)
+		(size 12.7 10.16)
 		(fields_autoplaced yes)
 		(stroke
@@
 		)
 		(property "Sheetname" "gsm"
-			(at 25.4 104.6984 0)
+			(at 27.94 98.3484 0)
 			(effects
 				(font
@@
 		)
 		(property "Sheetfile" "gsm.kicad_sch"
-			(at 25.4 119.9646 0)
+			(at 27.94 109.8046 0)
 			(effects
 				(font
@@
 			)
 		)
+		(pin "DTR" input
+			(at 40.64 100.33 0)
+			(effects
+				(font
+					(size 1.27 1.27)
+				)
+				(justify right)
+			)
+		)
+		(pin "RX" input
+			(at 40.64 102.87 0)
+			(effects
+				(font
+					(size 1.27 1.27)
+				)
+				(justify right)
+			)
+		)
+		(pin "TX" input
+			(at 40.64 105.41 0)
+			(effects
+				(font
+					(size 1.27 1.27)
+				)
+				(justify right)
+			)
+		)
+		(pin "PWRKEY" input
+			(at 40.64 107.95 0)
+			(effects
+				(font
+					(size 1.27 1.27)
+				)
+				(justify right)
+			)
+		)
 		(instances
 			(project "Phone"
@@
 	)
 	(sheet
-		(at 22.86 140.97)
+		(at 27.94 114.3)
 		(size 12.7 10.16)
 		(fields_autoplaced yes)
@@
 		)
 		(property "Sheetname" "GPS_Module"
-			(at 22.86 140.2584 0)
+			(at 27.94 113.5884 0)
 			(effects
 				(font
@@
 		)
 		(property "Sheetfile" "GPS_Module.kicad_sch"
-			(at 22.86 151.7146 0)
+			(at 27.94 125.0446 0)
 			(effects
 				(font
@@
 		)
 		(pin "TX" input
-			(at 35.56 146.05 0)
+			(at 40.64 119.38 0)
 			(effects
 				(font
@@
 		)
 		(pin "On{slash}Off" input
-			(at 35.56 148.59 0)
+			(at 40.64 121.92 0)
 			(effects
 				(font
@@
 		)
 		(pin "RX" input
-			(at 35.56 143.51 0)
+			(at 40.64 116.84 0)
 			(effects
 				(font
@@
 				)
 			)
+		)
+	)
+	(sheet
+		(at 24.13 129.54)
+		(size 16.51 26.67)
+		(fields_autoplaced yes)
+		(stroke
+			(width 0.1524)
+			(type solid)
+		)
+		(fill
+			(color 0 0 0 0.0000)
+		)
+		(property "Sheetname" "eink Display"
+			(at 24.13 128.8284 0)
+			(effects
+				(font
+					(size 1.27 1.27)
+				)
+				(justify left bottom)
+			)
+		)
+		(property "Sheetfile" "display.kicad_sch"
+			(at 24.13 156.7946 0)
+			(effects
+				(font
+					(size 1.27 1.27)
+				)
+				(justify left top)
+			)
+		)
+		(pin "D-SDA" input
+			(at 40.64 130.81 0)
+			(effects
+				(font
+					(size 1.27 1.27)
+				)
+				(justify right)
+			)
+		)
+		(pin "D-Data{slash}Command" input
+			(at 40.64 133.35 0)
+			(effects
+				(font
+					(size 1.27 1.27)
+				)
+				(justify right)
+			)
+		)
+		(pin "D-CS" input
+			(at 40.64 135.89 0)
+			(effects
+				(font
+					(size 1.27 1.27)
+				)
+				(justify right)
+			)
+		)
+		(pin "D-SCL" input
+			(at 40.64 138.43 0)
+			(effects
+				(font
+					(size 1.27 1.27)
+				)
+				(justify right)
+			)
+		)
+		(pin "D-BUSY" input
+			(at 40.64 140.97 0)
+			(effects
+				(font
+					(size 1.27 1.27)
+				)
+				(justify right)
+			)
+		)
+		(pin "D-RES" input
+			(at 40.64 143.51 0)
+			(effects
+				(font
+					(size 1.27 1.27)
+				)
+				(justify right)
+			)
+		)
+		(pin "T-SCL" input
+			(at 40.64 146.05 0)
+			(effects
+				(font
+					(size 1.27 1.27)
+				)
+				(justify right)
+			)
+		)
+		(pin "T-RST" input
+			(at 40.64 148.59 0)
+			(effects
+				(font
+					(size 1.27 1.27)
+				)
+				(justify right)
+			)
+		)
+		(pin "T-INT" input
+			(at 40.64 151.13 0)
+			(effects
+				(font
+					(size 1.27 1.27)
+				)
+				(justify right)
+			)
+		)
+		(pin "T-SDA" input
+			(at 40.64 153.67 0)
+			(effects
+				(font
+					(size 1.27 1.27)
+				)
+				(justify right)
+			)
+		)
+		(instances
+			(project "Phone"
+				(path "/3772f4af-284f-4c8c-b34e-39c18861d7c2"
+					(page "5")
+				)
+			)

Commit message: phone design is done abendoning projekt
Parts:
- removed C4: 1nF, Capacitor_SMD:C_1206_3216Metric, symbol Device:C
- removed F1: 2A PTC, Fuse:Fuse_1206_3216Metric_Pad1.42x1.75mm_HandSolder, symbol Device:Fuse
- removed J3: USB_C_Receptacle_USB2.0_16P, Connector_USB:USB_C_Receptacle_HRO_TYPE-C-31-M-12, symbol Connector:USB_C_Receptacle_USB2.0_16P
- removed R6, R7: 5k1, Resistor_SMD:R_1206_3216Metric, symbol Device:R
- removed R8: 1M, Resistor_SMD:R_1206_3216Metric, symbol Device:R
- removed U2: USBLC6-2SC6, Package_TO_SOT_SMD:SOT-23-6, symbol Power_Protection:USBLC6-2SC6
- added H3, H4, H5: MountingHole, MountingHole:MountingHole_3.2mm_M3, symbol Mechanical:MountingHole
- U1: footprint RF_Module:ESP32-S3-WROOM-1 -> RF_Module:ESP32-S3-WROOM-1U
Connections:
- net GND: no longer S1.4 (NO_2)
- net GPS_Module/On/Off: now also U1.4 (IO4)
- net GPS_Module/RX: now also U1.5 (IO5)
- net GPS_Module/TX: now also U1.6 (IO6)
- net eink Display/D-BUSY: now also U1.18 (IO10)
- net eink Display/D-CS: now also U1.21 (IO13)
- net eink Display/D-Data/Command: now also U1.20 (IO12)
- net eink Display/D-RES: now also U1.19 (IO11)
- net eink Display/D-SCL: now also U1.22 (IO14)
- net eink Display/T-RST: now also U1.12 (IO8)
- net eink Display/T-SDA: now also U1.17 (IO9)
- net gsm/DTR: now also U1.7 (IO7)
- net gsm/RX: now also U1.8 (IO15)
- net gsm/TX: now also U1.9 (IO16)
- net USBC/D+: now reaches U1.14 (IO20)
- net USBC/D-: now reaches U1.13 (IO19)
- net GSM-PKey: now reaches U1.10 (IO17)
- net T-INT: now reaches U1.11 (IO18)
- net T-SCL: now reaches U1.15 (IO3)
Other:
- added sheet BAT (BAT.kicad_sch)
- added sheet BoostConverter (BoostConverter.kicad_sch)
- added sheet USBC (USBC.kicad_sch)
- moved on the sheet: S1
