File: Hardware/Phone/GPS_Module.kicad_sch (KiCad schematic)
At the start: 4 parts, among them J4 Conn_Coaxial

Commit message: added doku. Abendoning Projekt
Parts:
- U4: value ~ -> ATGM336H-5N31
Changed lines of the file:
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@@
 			)
 		)
-		(property "Value" "~"
+		(property "Value" "ATGM336H-5N31"
 			(at 138.43 80.01 0)
 			(effects
